File: pcb/jm-daj.kicad_pcb (KiCad board)
At the start: 2 copper layers, 142 parts, among them J1 OLED_128x64, U1 nRF52840

Commit message: Finish matrix
Parts:
- removed D61, D62, D63, D64, D65, D66, D67, D68, D69, D70: Diode, ScottoKeebs_Components:Diode_SOD-123
- removed S61, S62, S63, S64, S65, S66, S67, S68, S69, S70: Keyswitch, ScottoKeebs_Hotswap:Hotswap_MX_1.00u
- added H1: Mounting_Hole, ScottoKeebs_Stabilizer:Stabilizer_MX_2.00u, F.Cu at (203.7, 130.3)
- added H2: Mounting_Hole, ScottoKeebs_Stabilizer:Stabilizer_MX_2.00u, F.Cu at (241.8, 130.4)
- added SW1: SW_Push, Button_Switch_THT:SW_Push_2P2T_Vertical_E-Switch_800UDP8P1A1M6, F.Cu at (219.4, 108.6)
- added U2: USBLC6-2SC6, Package_TO_SOT_SMD:SOT-23-6, F.Cu at (233.3, 49.8)
- D1, D10, D11, D12, D13, D14, D15, D16, D17, D18, D19, D2, D20, D21, D22, D23, D24, D25, D26, D27, D28, D29, D3, D30, D31, D32, D33, D34, D35, D36, D37, D38, D39, D4, D40, D41, D42, D43, D44, D45, D46, D47, D48, D49, D5, D50, D51, D52, D53, D54, D55, D56, D57, D58, D59, D6, D60, D7, D8, D9: moved to B.Cu
- S54, S55: footprint ScottoKeebs_Hotswap:Hotswap_MX_1.00u -> ScottoKeebs_Hotswap:Hotswap_MX_2.00u
- U1: value nRF52840 -> MDBT50Q-1MV2; footprint Package_DFN_QFN:Nordic_AQFN-73-1EP_7x7mm_P0.5mm -> RF_Module:Raytac_MDBT50Q
- moved S10 282.1 mm to (308.6, 54.7)
- moved S12 278.6 mm to (346.7, 54.7)
- moved S24 261.9 mm to (346.7, 73.7)
- moved S11 260.5 mm to (327.6, 54.7)
- moved S9 258.4 mm to (289.5, 54.7)
- moved S36 245.7 mm to (346.7, 92.8)
- moved S23 243.1 mm to (327.6, 73.7)
- moved S8 234.9 mm to (270.5, 54.7)
- moved S48 230.3 mm to (346.7, 111.8)
- moved S35 226.2 mm to (327.6, 92.8)
- moved S22 225.4 mm to (308.6, 73.7)
- moved S20 224.5 mm to (270.5, 73.7)
- moved S60 215.7 mm to (346.7, 130.9)
- moved S7 211.7 mm to (251.4, 54.7)
- moved S47 209.9 mm to (327.6, 111.8)
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Connections:
- D1 pad 1: unconnected-(D1-K-Pad1) -> Row 0
- D10 pad 1: unconnected-(D10-K-Pad1) -> Row 0
- D11 pad 1: unconnected-(D11-K-Pad1) -> Row 0
- D12 pad 1: unconnected-(D12-K-Pad1) -> Row 0
- D13 pad 1: unconnected-(D13-K-Pad1) -> Row 1
- D14 pad 1: unconnected-(D14-K-Pad1) -> Row 1
- D15 pad 1: unconnected-(D15-K-Pad1) -> Row 1
- D16 pad 1: unconnected-(D16-K-Pad1) -> Row 1
- D17 pad 1: unconnected-(D17-K-Pad1) -> Row 1
- D18 pad 1: unconnected-(D18-K-Pad1) -> Row 1
- D19 pad 1: unconnected-(D19-K-Pad1) -> Row 1
- D2 pad 1: unconnected-(D2-K-Pad1) -> Row 0
- D20 pad 1: unconnected-(D20-K-Pad1) -> Row 1
- D21 pad 1: unconnected-(D21-K-Pad1) -> Row 1
- D22 pad 1: unconnected-(D22-K-Pad1) -> Row 1
- D23 pad 1: unconnected-(D23-K-Pad1) -> Row 1
- D24 pad 1: unconnected-(D24-K-Pad1) -> Row 1
- D25 pad 1: unconnected-(D25-K-Pad1) -> Row 2
- D26 pad 1: unconnected-(D26-K-Pad1) -> Row 2
- D27 pad 1: unconnected-(D27-K-Pad1) -> Row 2
- D28 pad 1: unconnected-(D28-K-Pad1) -> Row 2
- D29 pad 1: unconnected-(D29-K-Pad1) -> Row 2
- D3 pad 1: unconnected-(D3-K-Pad1) -> Row 0
- D30 pad 1: unconnected-(D30-K-Pad1) -> Row 2
- D31 pad 1: unconnected-(D31-K-Pad1) -> Row 2
- D32 pad 1: unconnected-(D32-K-Pad1) -> Row 2
- D33 pad 1: unconnected-(D33-K-Pad1) -> Row 2
- D34 pad 1: unconnected-(D34-K-Pad1) -> Row 2
- D35 pad 1: unconnected-(D35-K-Pad1) -> Row 2
- D36 pad 1: unconnected-(D36-K-Pad1) -> Row 2
- D37 pad 1: unconnected-(D37-K-Pad1) -> Row 3
- D38 pad 1: unconnected-(D38-K-Pad1) -> Row 3
- D39 pad 1: unconnected-(D39-K-Pad1) -> Row 3
- D4 pad 1: unconnected-(D4-K-Pad1) -> Row 0
- D40 pad 1: unconnected-(D40-K-Pad1) -> Row 3
- D41 pad 1: unconnected-(D41-K-Pad1) -> Row 3
- D42 pad 1: unconnected-(D42-K-Pad1) -> Row 3
- D43 pad 1: unconnected-(D43-K-Pad1) -> Row 3
- D44 pad 1: unconnected-(D44-K-Pad1) -> Row 3
- D45 pad 1: unconnected-(D45-K-Pad1) -> Row 3
- D46 pad 1: unconnected-(D46-K-Pad1) -> Row 3
- D47 pad 1: unconnected-(D47-K-Pad1) -> Row 3
- D48 pad 1: unconnected-(D48-K-Pad1) -> Row 3
- D49 pad 1: unconnected-(D49-K-Pad1) -> Row 4
- D5 pad 1: unconnected-(D5-K-Pad1) -> Row 0
- D50 pad 1: unconnected-(D50-K-Pad1) -> Row 4
- D51 pad 1: unconnected-(D51-K-Pad1) -> Row 4
- D52 pad 1: unconnected-(D52-K-Pad1) -> Row 4
- D53 pad 1: unconnected-(D53-K-Pad1) -> Row 4
- D54 pad 1: unconnected-(D54-K-Pad1) -> Row 4
- D55 pad 1: unconnected-(D55-K-Pad1) -> Row 4
- D56 pad 1: unconnected-(D56-K-Pad1) -> Row 4
- D57 pad 1: unconnected-(D57-K-Pad1) -> Row 4
- D58 pad 1: unconnected-(D58-K-Pad1) -> Row 4
- D59 pad 1: unconnected-(D59-K-Pad1) -> Row 4
- D6 pad 1: unconnected-(D6-K-Pad1) -> Row 0
- D60 pad 1: unconnected-(D60-K-Pad1) -> Row 4
- D7 pad 1: unconnected-(D7-K-Pad1) -> Row 0
- D8 pad 1: unconnected-(D8-K-Pad1) -> Row 0
- D9 pad 1: unconnected-(D9-K-Pad1) -> Row 0
- J1 pad 1: unconnected-(J1-GND-Pad1) -> GND
- J1 pad 2: unconnected-(J1-VCC-Pad2) -> +3.3V
- J1 pad 3: unconnected-(J1-SCL-Pad3) -> Display Clock
- J1 pad 4: unconnected-(J1-SDA-Pad4) -> Display Data
- S1 pad 1: unconnected-(S1-Pad1) -> Column 0
- S10 pad 1: unconnected-(S10-Pad1) -> Column 9
- S11 pad 1: unconnected-(S11-Pad1) -> Column 10
- S12 pad 1: unconnected-(S12-Pad1) -> Column 11
- S13 pad 1: unconnected-(S13-Pad1) -> Column 0
- S14 pad 1: unconnected-(S14-Pad1) -> Column 1
- S15 pad 1: unconnected-(S15-Pad1) -> Column 2
- S16 pad 1: unconnected-(S16-Pad1) -> Column 3
- S17 pad 1: unconnected-(S17-Pad1) -> Column 4
- S18 pad 1: unconnected-(S18-Pad1) -> Column 5
- S19 pad 1: unconnected-(S19-Pad1) -> Column 6
- S2 pad 1: unconnected-(S2-Pad1) -> Column 1
- S20 pad 1: unconnected-(S20-Pad1) -> Column 7
- S21 pad 1: unconnected-(S21-Pad1) -> Column 8
- S22 pad 1: unconnected-(S22-Pad1) -> Column 9
- S23 pad 1: unconnected-(S23-Pad1) -> Column 10
- S24 pad 1: unconnected-(S24-Pad1) -> Column 11
- S25 pad 1: unconnected-(S25-Pad1) -> Column 0
- S26 pad 1: unconnected-(S26-Pad1) -> Column 1
- S27 pad 1: unconnected-(S27-Pad1) -> Column 2
- S28 pad 1: unconnected-(S28-Pad1) -> Column 3
- S29 pad 1: unconnected-(S29-Pad1) -> Column 4
- S3 pad 1: unconnected-(S3-Pad1) -> Column 2
- S30 pad 1: unconnected-(S30-Pad1) -> Column 5
- S31 pad 1: unconnected-(S31-Pad1) -> Column 6
- S32 pad 1: unconnected-(S32-Pad1) -> Column 7
- S33 pad 1: unconnected-(S33-Pad1) -> Column 8
- S34 pad 1: unconnected-(S34-Pad1) -> Column 9
- S35 pad 1: unconnected-(S35-Pad1) -> Column 10
- S36 pad 1: unconnected-(S36-Pad1) -> Column 11
- S37 pad 1: unconnected-(S37-Pad1) -> Column 0
- S38 pad 1: unconnected-(S38-Pad1) -> Column 1
- S39 pad 1: unconnected-(S39-Pad1) -> Column 2
- S4 pad 1: unconnected-(S4-Pad1) -> Column 3
- S40 pad 1: unconnected-(S40-Pad1) -> Column 3
- S41 pad 1: unconnected-(S41-Pad1) -> Column 4
- S42 pad 1: unconnected-(S42-Pad1) -> Column 5
- S43 pad 1: unconnected-(S43-Pad1) -> Column 6
- S44 pad 1: unconnected-(S44-Pad1) -> Column 7
- S45 pad 1: unconnected-(S45-Pad1) -> Column 8
- S46 pad 1: unconnected-(S46-Pad1) -> Column 9
- S47 pad 1: unconnected-(S47-Pad1) -> Column 10
- S48 pad 1: unconnected-(S48-Pad1) -> Column 11
- S49 pad 1: unconnected-(S49-Pad1) -> Column 0
- S5 pad 1: unconnected-(S5-Pad1) -> Column 4
- S50 pad 1: unconnected-(S50-Pad1) -> Column 1
- S51 pad 1: unconnected-(S51-Pad1) -> Column 2
- S52 pad 1: unconnected-(S52-Pad1) -> Column 3
- S53 pad 1: unconnected-(S53-Pad1) -> Column 4
- S54 pad 1: unconnected-(S54-Pad1) -> Column 5
- S55 pad 1: unconnected-(S55-Pad1) -> Column 6
- S56 pad 1: unconnected-(S56-Pad1) -> Column 7
- S57 pad 1: unconnected-(S57-Pad1) -> Column 8
- S58 pad 1: unconnected-(S58-Pad1) -> Column 9
- S59 pad 1: unconnected-(S59-Pad1) -> Column 10
- S6 pad 1: unconnected-(S6-Pad1) -> Column 5
- S60 pad 1: unconnected-(S60-Pad1) -> Column 11
- S7 pad 1: unconnected-(S7-Pad1) -> Column 6
- S8 pad 1: unconnected-(S8-Pad1) -> Column 7
- S9 pad 1: unconnected-(S9-Pad1) -> Column 8
Routing:
- net Row 4: track 0.00 -> 262.6 mm
- net Row 2: track 0.00 -> 247.7 mm
- net Row 3: track 0.00 -> 247.7 mm
- net Row 1: track 0.00 -> 247.7 mm
- net Row 0: track 0.00 -> 247.4 mm
- net Column 6: track 0.00 -> 101.8 mm, vias 0 -> 5
- net Column 5: track 0.00 -> 94.9 mm, vias 0 -> 5
- net Column 1: track 0.00 -> 93.5 mm, vias 0 -> 5
- net Column 8: track 0.00 -> 93.4 mm, vias 0 -> 5
- net Column 7: track 0.00 -> 93.4 mm, vias 0 -> 5
- net Column 9: track 0.00 -> 93.4 mm, vias 0 -> 5
- net Column 3: track 0.00 -> 93.4 mm, vias 0 -> 5
- net Column 4: track 0.00 -> 93.4 mm, vias 0 -> 5
- net Column 2: track 0.00 -> 93.4 mm, vias 0 -> 5
- net Column 11: track 0.00 -> 93.4 mm, vias 0 -> 5
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Other:
- board outline added: 274.1 x 100.4 mm
