File: pcb/jm-daj.kicad_sch (KiCad schematic)
At the start: 0 parts

Commit message: Update schema and add ScottoKicad addons
Parts:
- added C1: 1.0uf, symbol Device:C
- added D1, D10, D11, D12, D13, D14, D15, D16, D17, D18, D19, D2, D20, D23, D24, D25, D26, D27, D28, D29, D3, D30, D31, D32, D33, D34, D37, D38, D39, D4, D40, D41, D42, D43, D44, D45, D46, D47, D48, D5, D51, D52, D53, D54, D55, D56, D57, D58, D59, D6, D60, D61, D62, D65, D66, D67, D68, D69, D70, D9: Diode, ScottoKeebs_Components:Diode_SOD-123, symbol ScottoKeebs:Placeholder_Diode
- added J1: OLED_128x64, ScottoKeebs_Components:OLED_128x64, symbol ScottoKeebs:OLED_128x64
- added J2: USB_C_Receptacle_USB2.0_16P, symbol Connector:USB_C_Receptacle_USB2.0_16P
- added S1, S10, S11, S12, S13, S14, S15, S16, S17, S18, S19, S2, S20, S23, S24, S25, S26, S27, S28, S29, S3, S30, S31, S32, S33, S34, S37, S38, S39, S4, S40, S41, S42, S43, S44, S45, S46, S47, S48, S5, S51, S52, S53, S54, S55, S56, S57, S58, S59, S6, S60, S61, S62, S65, S66, S67, S68, S69, S70, S9: Keyswitch, ScottoKeebs_Hotswap:Hotswap_MX_1.00u, symbol ScottoKeebs:Placeholder_Keyswitch
- added U1: nRF52840, Package_DFN_QFN:Nordic_AQFN-73-1EP_7x7mm_P0.5mm, symbol MCU_Nordic:nRF52840
Connections:
- new net: D43.2 (A), S43.2
- new net: D11.2 (A), S11.2
- new net: D19.2 (A), S19.2
- new net: D20.2 (A), S20.2
- new net: D24.2 (A), S24.2
- new net: C1.2, U1.A18 (DEC2)
- new net: D12.2 (A), S12.2
- new net: D55.2 (A), S55.2
- new net: D42.2 (A), S42.2
- new net: D40.2 (A), S40.2
- new net: D67.2 (A), S67.2
- new net: D4.2 (A), S4.2
- new net: D26.2 (A), S26.2
- new net: D30.2 (A), S30.2
- new net: D1.2 (A), S1.2
- new net: D17.2 (A), S17.2
- new net: D70.2 (A), S70.2
- new net: D37.2 (A), S37.2
- new net: D33.2 (A), S33.2
- new net: D28.2 (A), S28.2
- new net: D9.2 (A), S9.2
- new net: D48.2 (A), S48.2
- new net: D41.2 (A), S41.2
- new net: D38.2 (A), S38.2
- new net: D59.2 (A), S59.2
- new net: D25.2 (A), S25.2
- new net: D6.2 (A), S6.2
- new net: D39.2 (A), S39.2
- new net: D18.2 (A), S18.2
- new net: D52.2 (A), S52.2
- new net: D62.2 (A), S62.2
- new net: D61.2 (A), S61.2
- new net: D29.2 (A), S29.2
- new net: D34.2 (A), S34.2
- new net: D32.2 (A), S32.2
- new net: J2.A1 (GND), J2.A12 (GND), J2.B1 (GND), J2.B12 (GND)
- new net: J2.A4 (VBUS), J2.A9 (VBUS), J2.B4 (VBUS), J2.B9 (VBUS)
- new net: D10.2 (A), S10.2
- new net: D58.2 (A), S58.2
- new net: D57.2 (A), S57.2
- new net: D46.2 (A), S46.2
- new net: D23.2 (A), S23.2
- new net: D15.2 (A), S15.2
- new net: D44.2 (A), S44.2
- new net: D45.2 (A), S45.2
- new net: D27.2 (A), S27.2
- new net: D31.2 (A), S31.2
- new net: D56.2 (A), S56.2
- new net: D16.2 (A), S16.2
- new net: D65.2 (A), S65.2
- new net: D60.2 (A), S60.2
- new net: D66.2 (A), S66.2
- new net: D5.2 (A), S5.2
- new net: D68.2 (A), S68.2
- new net: D54.2 (A), S54.2
- new net: D2.2 (A), S2.2
- new net: D53.2 (A), S53.2
- new net: D51.2 (A), S51.2
- new net: D13.2 (A), S13.2
- new net: D47.2 (A), S47.2
- new net: D69.2 (A), S69.2
- new net: D3.2 (A), S3.2
- new net: D14.2 (A), S14.2
- new net +3.3V: J1.2 (VCC), U1.A22 (VDD), U1.AD14 (VDD), U1.AD2 (VBUS), U1.AD23 (VDD), U1.B1 (VDD), U1.W1 (VDD), U1.Y2 (VDDH)
- new net Battery Reading: U1.J1 (AIN2/P0.04)
- new net Column 0: S1.1, S15.1, S29.1, S43.1, S57.1, U1.AC9 (P0.14)
- new net Column 1: S16.1, S2.1, S30.1, S44.1, S58.1, U1.AD10 (P0.15)
- new net Column 10: S13.1, S27.1, S41.1, S55.1, S69.1, U1.AC21 (P0.25)
- new net Column 11: S14.1, S28.1, S42.1, S56.1, S70.1, U1.G1 (P0.26)
- new net Column 2: S17.1, S3.1, S31.1, S45.1, S59.1, U1.AC11 (P0.16)
- new net Column 3: S18.1, S32.1, S4.1, S46.1, S60.1, U1.AD12 (P0.17)
- new net Column 4: S19.1, S33.1, S47.1, S5.1, S61.1, U1.AC15 (P0.19)
- new net Column 5: S20.1, S34.1, S48.1, S6.1, S62.1, U1.AD16 (P0.20)
- new net Column 6: S23.1, S37.1, S51.1, S65.1, S9.1, U1.AC17 (P0.21)
- new net Column 7: S10.1, S24.1, S38.1, S52.1, S66.1, U1.AD18 (P0.22)
- new net Column 8: S11.1, S25.1, S39.1, S53.1, S67.1, U1.AC19 (P0.23)
- new net Column 9: S12.1, S26.1, S40.1, S54.1, S68.1, U1.AD20 (P0.24)
- new net Cut off power to VCC: U1.AD8 (P0.13)
- new net Display Clock: J1.3 (SCL), U1.B13 (AIN1/P0.03)
- new net Display Data: J1.4 (SDA), U1.A12 (AIN0/P0.02)
- new net GND: C1.1, J1.1 (GND), U1.B7 (VSS), U1.EP (VSS), U1.F23 (VSS_PA)
- new net Row 0: D1.1 (K), D10.1 (K), D11.1 (K), D12.1 (K), D13.1 (K), D14.1 (K), D2.1 (K), D3.1 (K), D4.1 (K), D5.1 (K), D6.1 (K), D9.1 (K), U1.Y23 (P1.01)
- new net Row 1: D15.1 (K), D16.1 (K), D17.1 (K), D18.1 (K), D19.1 (K), D20.1 (K), D23.1 (K), D24.1 (K), D25.1 (K), D26.1 (K), D27.1 (K), D28.1 (K), U1.W24 (P1.02)
- new net Row 2: D29.1 (K), D30.1 (K), D31.1 (K), D32.1 (K), D33.1 (K), D34.1 (K), D37.1 (K), D38.1 (K), D39.1 (K), D40.1 (K), D41.1 (K), D42.1 (K), U1.V23 (P1.03)
- new net Row 3: D43.1 (K), D44.1 (K), D45.1 (K), D46.1 (K), D47.1 (K), D48.1 (K), D51.1 (K), D52.1 (K), D53.1 (K), D54.1 (K), D55.1 (K), D56.1 (K), U1.U24 (P1.04)
- new net Row 4: D57.1 (K), D58.1 (K), D59.1 (K), D60.1 (K), D61.1 (K), D62.1 (K), D65.1 (K), D66.1 (K), D67.1 (K), D68.1 (K), D69.1 (K), D70.1 (K), U1.T23 (P1.05)
- new net USB D+: U1.AD6 (D+)
- new net USB D-: U1.AD4 (D-)

Commit message: Finish matrix
Parts:
- removed U1: nRF52840, Package_DFN_QFN:Nordic_AQFN-73-1EP_7x7mm_P0.5mm, symbol MCU_Nordic:nRF52840
- added C2, C3, C4: C, symbol Device:C
- added H1, H2: Mounting_Hole, ScottoKeebs_Stabilizer:Stabilizer_MX_2.00u, symbol ScottoKeebs:Placeholder_Mounting_Hole
- added L1: L, symbol Device:L
- added R1, R2: 5.1k, symbol Device:R
- added R3, R4, R5: R, symbol Device:R
- added SW1: SW_Push, Button_Switch_THT:SW_Push_2P2T_Vertical_E-Switch_800UDP8P1A1M6, symbol Switch:SW_Push
- added U1: MDBT50Q-1MV2, RF_Module:Raytac_MDBT50Q, symbol RF_Module:MDBT50Q-1MV2
- added U2: USBLC6-2SC6, Package_TO_SOT_SMD:SOT-23-6, symbol Power_Protection:USBLC6-2SC6
- added U3: TPS62822DLC, Package_SON:Texas_VSON-HR-8_1.5x2mm_P0.5mm, symbol Regulator_Switching:TPS62822DLC
- C1: value 1.0uf -> C
- S54: renamed from S62; footprint ScottoKeebs_Hotswap:Hotswap_MX_1.00u -> ScottoKeebs_Hotswap:Hotswap_MX_2.00u
- S55: renamed from S65; footprint ScottoKeebs_Hotswap:Hotswap_MX_1.00u -> ScottoKeebs_Hotswap:Hotswap_MX_2.00u
- renumbered D12 to D10, D13 to D11, D14 to D12, D15 to D13, D16 to D14, D17 to D15, D18 to D16, D19 to D17, D20 to D18, D23 to D19, D24 to D20, D25 to D21, D26 to D22, D27 to D23, D28 to D24, D29 to D25, D30 to D26, D31 to D27, D32 to D28, D33 to D29, D34 to D30, D37 to D31, D38 to D32, D39 to D33, D40 to D34, D41 to D35, D42 to D36, D43 to D37, D44 to D38, D45 to D39, D46 to D40, D47 to D41, D48 to D42, D51 to D43, D52 to D44, D53 to D45, D54 to D46, D55 to D47, D56 to D48, D57 to D49, D58 to D50, D59 to D51, D60 to D52, D61 to D53, D62 to D54, D65 to D55, D66 to D56, D67 to D57, D68 to D58, D69 to D59, D70 to D60, D9 to D7, D10 to D8, D11 to D9, S12 to S10, S13 to S11, S14 to S12, S15 to S13, S16 to S14, S17 to S15, S18 to S16, S19 to S17, S20 to S18, S23 to S19, S24 to S20, S25 to S21, S26 to S22, S27 to S23, S28 to S24, S29 to S25, S30 to S26, S31 to S27, S32 to S28, S33 to S29, S34 to S30, S37 to S31, S38 to S32, S39 to S33, S40 to S34, S41 to S35, S42 to S36, S43 to S37, S44 to S38, S45 to S39, S46 to S40, S47 to S41, S48 to S42, S51 to S43, S52 to S44, S53 to S45, S54 to S46, S55 to S47, S56 to S48, S57 to S49, S58 to S50, S59 to S51, S60 to S52, S61 to S53, S66 to S56, S67 to S57, S68 to S58, S69 to S59, S70 to S60, S9 to S7, S10 to S8, S11 to S9
Connections:
- net Column 0: now also U1.8 (P1.15)
- net Column 1: now also U1.10 (P0.29)
- net Column 10: now also U1.57 (P1.06)
- net Column 11: now also U1.59 (P1.05)
- net Column 2: now also U1.12 (P0.31)
- net Column 3: now also U1.14 (P0.30)
- net Column 4: now also U1.13 (P0.28)
- net Column 5: now also U1.11 (P0.02)
- net Column 6: now also U1.9 (P0.03)
- net Column 7: now also U1.60 (P1.03)
- net Column 8: now also U1.58 (P1.07)
- net Column 9: now also U1.56 (P1.04)
- net GND: now also J2.A1 (GND), J2.A12 (GND), J2.B1 (GND), J2.B12 (GND), J2.S1 (SHIELD), C2.2, C3.2, C4.2, R1.2, R2.2, R4.2, R5.2, SW1.2, U1.1 (GND), U1.15 (GND), U1.2 (GND), U1.33 (GND), U1.55 (GND), U2.2 (GND), U3.3 (AGND), U3.5 (PGND); no longer C1.1
- net Row 0: now also U1.7 (P1.14)
- net Row 1: now also U1.6 (P1.13)
- net Row 2: now also U1.5 (P1.12)
- net Row 3: now also U1.4 (P1.11)
- net Row 4: now also U1.3 (P1.10)
- net at C1.2: now also R3.2, R4.1, U3.2 (FB)
- net VBUS: now reaches J2.A4 (VBUS), J2.A9 (VBUS), J2.B4 (VBUS), J2.B9 (VBUS)
- net VBUS: now also U1.32 (VBUS), U2.5 (VBUS)
- net at J2.A5 (CC1): now also R1.1
- net D+ Connection: now reaches J2.A6 (D+)
- net D+ Connection: now also J2.B6 (D+), U2.1 (I/O1)
- net D- Connection: now reaches J2.A7 (D-)
- net D- Connection: now also J2.B7 (D-), U2.6 (I/O1)
- net at J2.B5 (CC2): now also R2.1
- new net: SW1.1, U1.40 (P0.18)
- new net: U3.1 (EN), U3.7 (VIN)
- new net: L1.1, U3.6 (SW)
- new net 0.20: U1.44 (P0.20)
- new net 0.21: U1.43 (P0.21)
- new net 0.22: U1.46 (P0.22)
- new net 0.24: U1.48 (P0.24)
- new net 0.25: U1.49 (P0.25)
- new net BVOLT: U1.20 (P0.04)
- new net D+: U1.35 (D+), U2.3 (I/O2)
- new net D-: U1.34 (D-), U2.4 (I/O2)
- new net NFC1: U1.52 (P0.09)
- new net NFC2: U1.54 (P0.10)
- new net Power pin: U1.21 (P0.05)
- new net SWC: U1.53 (SWDCLK)
- new net SWD: U1.51 (SWDIO)
- new net VDD_NRF: C1.1, C2.1, L1.2, R3.1, U1.28 (VDD), U1.30 (VDDH)
- no-connect marks 0 -> 23
Other:
- moved on the sheet: D1, D10, D11, D12, D13, D14, D15, D16, D17, D18, D19, D2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
